File: backplane.sch (KiCad schematic (older format))
At the start: 34 parts, among them J1 I2C, J2 I2C, J3 SER, J4 PWR, J5 PWR, J6 FAN, J7 PPS, Q4 Q_NMOS_GSD, Q5 Q_PMOS_GSD, SW1 SW_Push, U1 Raspberry_Pi_2_3, U2 IC880A-SPI, U4 MP1584_MODULE, U5 MCP3425A0T-E/CH, U6 SHTC3

Commit message: modifikace pro FEI/VSB
Parts:
- added R6: R, Resistor_SMD:R_1206_3216Metric_Pad1.42x1.75mm_HandSolder, symbol backplane-rescue:R-backplane-rescue
- added U3: DHT11, Connector_PinHeader_2.54mm:PinHeader_1x04_P2.54mm_Vertical, symbol Sensor:DHT11
- added U7: LM2596_MODULE, regulators:LM2596_MODULE, symbol regulators:LM2596_MODULE
- C1, C3: footprint Capacitors_SMD:C_1206 -> Capacitor_SMD:C_1206_3216Metric_Pad1.42x1.75mm_HandSolder; symbol backplane-rescue:C -> backplane-rescue:C-backplane-rescue
- D1, D2, D3: footprint LEDs:LED_1206 -> LED_SMD:LED_1206_3216Metric_Pad1.42x1.75mm_HandSolder; symbol backplane-rescue:LED_Small -> backplane-rescue:LED_Small-backplane-rescue
- D4, D6: footprint DO214:DO-214AC -> Diode_SMD:D_2114_3652Metric; symbol backplane-rescue:D -> backplane-rescue:D-backplane-rescue
- D5: footprint DO214:DO-214AA -> Diode_SMD:D_2114_3652Metric; symbol backplane-rescue:D_Zener_Small -> backplane-rescue:D_Zener_Small-backplane-rescue
- F1: footprint Capacitors_SMD:C_1812 -> Capacitor_SMD:C_1812_4532Metric_Pad1.30x3.40mm_HandSolder; symbol backplane-rescue:Polyfuse_Small -> backplane-rescue:Polyfuse_Small-backplane-rescue
- J1, J2: symbol backplane-rescue:I2C_HEADER -> backplane-rescue:I2C_HEADER-backplane-rescue
- J3: symbol backplane-rescue:SERIAL_HEADER -> backplane-rescue:SERIAL_HEADER-backplane-rescue
- J4, J5: footprint Connectors_Terminal_Blocks:TerminalBlock_Pheonix_MPT-2.54mm_2pol -> TerminalBlock_Phoenix:TerminalBlock_Phoenix_MPT-0,5-2-2.54_1x02_P2.54mm_Horizontal; symbol backplane-rescue:PWR_HEADER -> backplane-rescue:PWR_HEADER-backplane-rescue
- J6: footprint headers:header_1x2_marked -> headers:header_1x2_unmarked; symbol backplane-rescue:FAN -> backplane-rescue:FAN-backplane-rescue
- J7: symbol backplane-rescue:Conn_01x01 -> backplane-rescue:Conn_01x01-backplane-rescue
- Q4: footprint TO_SOT_Packages_SMD:SOT-23 -> Package_TO_SOT_SMD:SOT-23; symbol backplane-rescue:Q_NMOS_GSD -> backplane-rescue:Q_NMOS_GSD-backplane-rescue
- Q5: footprint TO_SOT_Packages_SMD:SOT-23 -> Package_TO_SOT_SMD:SOT-23; symbol backplane-rescue:Q_PMOS_GSD -> backplane-rescue:Q_PMOS_GSD-backplane-rescue
- R1, R2, R3: footprint Resistors_SMD:R_1206 -> Resistor_SMD:R_1206_3216Metric_Pad1.42x1.75mm_HandSolder; symbol backplane-rescue:R-RESCUE-backplane -> backplane-rescue:R-RESCUE-backplane-backplane-rescue
- R10, R11, R12: footprint Resistors_SMD:R_0805 -> Resistor_SMD:R_0805_2012Metric_Pad1.15x1.40mm_HandSolder; symbol backplane-rescue:R -> backplane-rescue:R-backplane-rescue
- R13, R4, R5, R9: footprint Resistors_SMD:R_1206 -> Resistor_SMD:R_1206_3216Metric_Pad1.42x1.75mm_HandSolder; symbol backplane-rescue:R -> backplane-rescue:R-backplane-rescue
- SW1: symbol backplane-rescue:SW_Push -> backplane-rescue:SW_Push-backplane-rescue
- U1: footprint headers:Pin_Header_Straight_2x20_Pitch2.54mm -> Pin_Headers:Pin_Header_Straight_2x20; symbol backplane-rescue:Raspi_2_3 -> backplane-rescue:Raspi_2_3-backplane-rescue
- U2: symbol backplane-rescue:IC880A-SPI -> backplane-rescue:IC880A-SPI-backplane-rescue
- U4: symbol backplane-rescue:MP1584_MODULE -> backplane-rescue:MP1584_MODULE-backplane-rescue
- U5: footprint TO_SOT_Packages_SMD:SOT-23-6 -> Package_TO_SOT_SMD:SOT-23-6_Handsoldering; symbol backplane-rescue:MCP3425A0T-E_CH-RESCUE-backplane -> backplane-rescue:MCP3425A0T-E_CH-RESCUE-backplane-backplane-rescue
- U6: symbol backplane-rescue:SHTC3 -> backplane-rescue:SHTC3-backplane-rescue
Connections:
- net labels added: DHT_IO
- wire segments 185 -> 206
- no-connect marks 23 -> 22
Other:
- note added: "DHT22"
- note added: "The board includes a 5V\npower input/output\nconnector as well as a\nMP1584 or LM2596 \nstep-down voltage regulator\nfor 6.7-28V input."
- note removed: "The board includes a 5V\npower input/output\nconnector as well as a\nMP1584 step-down\nvoltage regulator for\n6.7-28V input."

Commit message: values in schematics moved into value field, generated BOM
Parts:
- C1: value C -> 100nF; C 100nF -> (none); shop (none) -> https://www.gme.cz/cks1206-100n-50v-x7r-10-yageo
- C3: value C -> 100nF; C 100nF -> (none)
- D4, D6: value D -> SS14
- D5: value D_TVS -> TVSD SMBJ5.0A
- F1: value Polyfuse -> PolySwitch (PTC)
- R10: value R -> 6.8kΩ; R 6.8kΩ -> (none)
- R11: value R -> 3.6kΩ; R 3.6kΩ -> (none)
- R12: value R -> 470Ω; R 470Ω -> (none)
- R13, R4, R5, R9: value R -> 10kΩ; R 10kΩ -> (none)
- R6: value R -> 4.7kΩ; R 4.7kΩ -> (none)
- U3: value DHT11 -> DHT22
Other:
- moved on the sheet: D6
Changed lines of the file:
@@
 P 3950 1250
 F 0 "C1" H 3950 1350 40  0000 L CNN
-F 1 "C" H 3956 1165 40  0000 L CNN
+F 1 "100nF" H 3956 1165 40  0000 L CNN
 F 2 "Capacitor_SMD:C_1206_3216Metric_Pad1.42x1.75mm_HandSolder" H 3988 1100 30  0001 C CNN
 F 3 "" H 3950 1250 60  0001 C CNN
-F 4 "100nF" V 3800 1250 60  0000 C CNN "C"
+F 4 "https://www.gme.cz/cks1206-100n-50v-x7r-10-yageo" H 3950 1250 50  0001 C CNN "shop"
 	1    3950 1250
 	0    1    1    0
@@
 U 1 1 589B82C4
 P 5150 1000
-F 0 "R4" V 5230 1000 40  0000 C CNN
-F 1 "R" V 5157 1001 40  0000 C CNN
+F 0 "R4" V 5050 1000 40  0000 C CNN
+F 1 "10kΩ" V 5157 1001 40  0000 C CNN
 F 2 "Resistor_SMD:R_1206_3216Metric_Pad1.42x1.75mm_HandSolder" V 5080 1000 30  0001 C CNN
 F 3 "" H 5150 1000 30  0000 C CNN
-F 4 "10kΩ" V 5050 1000 60  0000 C CNN "R"
 	1    5150 1000
 	0    1    1    0
@@
 U 1 1 589B831C
 P 5150 1250
-F 0 "R5" V 5230 1250 40  0000 C CNN
-F 1 "R" V 5157 1251 40  0000 C CNN
+F 0 "R5" V 5050 1250 40  0000 C CNN
+F 1 "10kΩ" V 5157 1251 40  0000 C CNN
 F 2 "Resistor_SMD:R_1206_3216Metric_Pad1.42x1.75mm_HandSolder" V 5080 1250 30  0001 C CNN
 F 3 "" H 5150 1250 30  0000 C CNN
-F 4 "10kΩ" V 5050 1250 60  0000 C CNN "R"
 	1    5150 1250
 	0    1    1    0
@@
 U 1 1 589CC7B2
 P 9950 5600
-F 0 "D4" H 9950 5700 50  0000 C CNN
-F 1 "D" H 9950 5500 50  0000 C CNN
+F 0 "D4" H 9950 5500 50  0000 C CNN
+F 1 "SS14" H 9950 5700 50  0000 C CNN
 F 2 "Diode_SMD:D_2114_3652Metric" H 9950 5600 50  0001 C CNN
 F 3 "" H 9950 5600 50  0001 C CNN
@@
 U 1 1 589F7FAA
 P 8700 1100
-F 0 "U4" H 9050 800 60  0000 C CNN
-F 1 "MP1584_MODULE" H 8700 1450 60  0000 C CNN
+F 0 "U4" H 8700 850 60  0000 C CNN
+F 1 "MP1584_MODULE" H 8700 1400 60  0000 C CNN
 F 2 "regulators:MP1584_MODULE_ZVEPOWER" H 8700 1100 60  0001 C CNN
 F 3 "" H 8700 1100 60  0001 C CNN
@@
 U 1 1 58A8FA09
 P 10350 6200
-F 0 "R9" V 10430 6200 50  0000 C CNN
-F 1 "R" V 10350 6200 50  0000 C CNN
+F 0 "R9" V 10250 6200 50  0000 C CNN
+F 1 "10kΩ" V 10350 6200 50  0000 C CNN
 F 2 "Resistor_SMD:R_1206_3216Metric_Pad1.42x1.75mm_HandSolder" V 10280 6200 50  0001 C CNN
 F 3 "" H 10350 6200 50  0000 C CNN
-F 4 "10kΩ" V 10250 6200 60  0000 C CNN "R"
 	1    10350 6200
 	0    1    1    0
@@
 P 10050 3800
 F 0 "U5" H 9650 4100 50  0000 L CNN
-F 1 "MCP3425A0T-E/CH" H 10150 4100 50  0000 L CNN
+F 1 "MCP3425A0T-E/CH" H 10150 3450 50  0000 L CNN
 F 2 "Package_TO_SOT_SMD:SOT-23-6_Handsoldering" H 10050 3800 50  0001 C CIN
 F 3 "" H 10050 3800 50  0000 C CNN
@@
 U 1 1 58F15A4C
 P 8950 3800
-F 0 "R11" V 9030 3800 50  0000 C CNN
-F 1 "R" V 8950 3800 50  0000 C CNN
+F 0 "R11" V 8850 3800 50  0000 C CNN
+F 1 "3.6kΩ" V 8950 3800 50  0000 C CNN
 F 2 "Resistor_SMD:R_0805_2012Metric_Pad1.15x1.40mm_HandSolder" V 8880 3800 50  0001 C CNN
 F 3 "" H 8950 3800 50  0000 C CNN
-F 4 "3.6kΩ" V 8850 3800 60  0000 C CNN "R"
 	1    8950 3800
 	1    0    0    -1
@@
 U 1 1 58F15AE0
 P 8950 3400
-F 0 "R10" V 9030 3400 50  0000 C CNN
-F 1 "R" V 8950 3400 50  0000 C CNN
+F 0 "R10" V 8850 3400 50  0000 C CNN
+F 1 "6.8kΩ" V 8950 3400 50  0000 C CNN
 F 2 "Resistor_SMD:R_0805_2012Metric_Pad1.15x1.40mm_HandSolder" V 8880 3400 50  0001 C CNN
 F 3 "" H 8950 3400 50  0000 C CNN
-F 4 "6.8kΩ" V 8850 3400 60  0000 C CNN "R"
 	1    8950 3400
 	1    0    0    -1
@@
 U 1 1 58F15B81
 P 8950 4200
-F 0 "R12" V 9030 4200 50  0000 C CNN
-F 1 "R" V 8950 4200 50  0000 C CNN
+F 0 "R12" V 8850 4200 50  0000 C CNN
+F 1 "470Ω" V 8950 4200 50  0000 C CNN
 F 2 "Resistor_SMD:R_0805_2012Metric_Pad1.15x1.40mm_HandSolder" V 8880 4200 50  0001 C CNN
 F 3 "" H 8950 4200 50  0000 C CNN
-F 4 "470Ω" V 8850 4200 60  0000 C CNN "R"
 	1    8950 4200
 	1    0    0    -1
@@
 U 1 1 58F17903
 P 9200 3800
-F 0 "C3" H 9200 3900 40  0000 L CNN
-F 1 "C" H 9206 3715 40  0000 L CNN
+F 0 "C3" H 9250 3700 40  0000 L CNN
+F 1 "100nF" H 9000 3900 40  0000 L CNN
 F 2 "Capacitor_SMD:C_1206_3216Metric_Pad1.42x1.75mm_HandSolder" H 9238 3650 30  0001 C CNN
 F 3 "" H 9200 3800 60  0001 C CNN
-F 4 "100nF" V 9050 3800 60  0000 C CNN "C"
 	1    9200 3800
 	-1   0    0    1
@@
 U 1 1 58F8FE37
 P 10800 1550
-F 0 "D5" H 10800 1640 50  0000 C CNN
-F 1 "D_TVS" H 10800 1460 50  0000 C CNN
+F 0 "D5" H 10800 1450 50  0000 C CNN
+F 1 "TVSD SMBJ5.0A" H 10800 1650 50  0000 C CNN
 F 2 "Diode_SMD:D_2114_3652Metric" V 10800 1550 50  0001 C CNN
 F 3 "" V 10800 1550 50  0001 C CNN
@@
 U 1 1 58F913C4
 P 10000 1100
-F 0 "F1" V 9900 1100 50  0000 C CNN
-F 1 "Polyfuse" V 10100 1100 50  0000 C CNN
+F 0 "F1" V 10100 1100 50  0000 C CNN
+F 1 "PolySwitch (PTC)" V 9900 1100 50  0000 C CNN
 F 2 "Capacitor_SMD:C_1812_4532Metric_Pad1.30x3.40mm_HandSolder" H 10050 900 50  0001 L CNN
 F 3 "" H 10000 1100 50  0001 C CNN
@@
 L backplane-rescue:D-backplane-rescue D6
 U 1 1 58F9565C
-P 8700 700
-F 0 "D6" H 8550 650 50  0000 C CNN
-F 1 "D" H 8800 650 50  0000 C CNN
-F 2 "Diode_SMD:D_2114_3652Metric" H 8700 700 50  0001 C CNN
-F 3 "" H 8700 700 50  0001 C CNN
-F 4 "Vishay SS14" H 8700 700 60  0001 C CNN "Model"
-	1    8700 700
+P 8700 650
+F 0 "D6" H 8550 700 50  0000 C CNN
+F 1 "SS14" H 8700 600 50  0000 C CNN
+F 2 "Diode_SMD:D_2114_3652Metric" H 8700 650 50  0001 C CNN
+F 3 "" H 8700 650 50  0001 C CNN
+F 4 "Vishay SS14" H 8700 650 60  0001 C CNN "Model"
+	1    8700 650
 	1    0    0    -1
 $EndComp
@@
 U 1 1 58F98D63
 P 10400 1200
-F 0 "Q5" V 10300 1250 50  0000 L CNN
-F 1 "Q_PMOS_GSD" V 10700 950 50  0000 L CNN
+F 0 "Q5" V 10650 1150 50  0000 L CNN
+F 1 "Q_PMOS_GSD" V 10250 1000 50  0000 L CNN
 F 2 "Package_TO_SOT_SMD:SOT-23" H 10600 1300 50  0001 C CNN
 F 3 "" H 10400 1200 50  0001 C CNN
@@
 P 10400 1700
 F 0 "R13" V 10480 1700 40  0000 C CNN
-F 1 "R" V 10400 1700 40  0000 C CNN
+F 1 "10kΩ" V 10400 1700 40  0000 C CNN
 F 2 "Resistor_SMD:R_1206_3216Metric_Pad1.42x1.75mm_HandSolder" V 10330 1700 30  0001 C CNN
 F 3 "" H 10400 1700 30  0000 C CNN
-F 4 "10kΩ" V 10300 1700 60  0000 C CNN "R"
 	1    10400 1700
 	-1   0    0    1
@@
 	8500 6200 8500 6250
 Wire Wire Line
-	8200 700  8550 700
-Wire Wire Line
-	8850 700  9200 700
-Wire Wire Line
 	9150 1100 9200 1100
 Wire Wire Line
@@
 Wire Wire Line
 	10950 2400 10950 2500
-Wire Wire Line
-	8200 700  8200 950
 Connection ~ 8200 1100
-Wire Wire Line
-	9200 700  9200 1100
 Connection ~ 9200 1100
 Wire Wire Line
@@
 P 1700 3050
 F 0 "U3" V 1333 3050 50  0000 C CNN
-F 1 "DHT11" V 1424 3050 50  0000 C CNN
+F 1 "DHT22" V 1424 3050 50  0000 C CNN
 F 2 "Connector_PinHeader_2.54mm:PinHeader_1x04_P2.54mm_Vertical" H 1850 3300 50  0001 C CNN
 F 3 "" H 1850 3300 50  0001 C CNN
@@
 P 2150 3200
 F 0 "R6" V 2230 3200 40  0000 C CNN
-F 1 "R" V 2157 3201 40  0000 C CNN
+F 1 "4.7kΩ" V 2157 3201 40  0000 C CNN
 F 2 "Resistor_SMD:R_1206_3216Metric_Pad1.42x1.75mm_HandSolder" V 2080 3200 30  0001 C CNN
 F 3 "" H 2150 3200 30  0000 C CNN
-F 4 "4.7kΩ" V 2050 3200 60  0000 C CNN "R"
 	1    2150 3200
 	-1   0    0    1
@@
 U 1 1 5D528ACB
 P 8700 1950
-F 0 "U7" H 8700 2337 60  0000 C CNN
-F 1 "LM2596_MODULE" H 8700 2231 60  0000 C CNN
+F 0 "U7" H 8700 2200 60  0000 C CNN
+F 1 "LM2596_MODULE" H 8700 1700 60  0000 C CNN
 F 2 "regulators:LM2596_MODULE" H 8700 1950 60  0001 C CNN
 F 3 "https://laskarduino.cz/step-down-menice/120003-step-down-menic-s-lm2596.html" H 8700 1950 60  0001 C CNN
@@
 	1    0    0    -1
 $EndComp
+Wire Wire Line
+	8200 650  8550 650
+Wire Wire Line
+	8200 650  8200 950
+Wire Wire Line
+	8850 650  9200 650
+Wire Wire Line
+	9200 650  9200 1100
 $EndSCHEMATC
