File: backplane.kicad_pcb (KiCad board)
At the start: 2 copper layers, 93.9 x 83.8 mm, 72 parts, among them J1 I2C, J2 I2C, J3 SER, J4 PWR, J5 PWR, J6 FAN, J7 PPS, Q4 Q_NMOS_GSD, Q5 Q_PMOS_GSD, SW1 SW_Push, U1 Raspberry_Pi_2_3, U2 IC880A-SPI, U4 MP1584_MODULE, U5 MCP3425A0T-E/CH, U6 SHTC3

Commit message: modifikace pro FEI/VSB
Parts:
- removed G***: LOGO, oshw-logos:OSHW_MASK_7MM
- removed the REF** at (124.0, 86.6)
- removed the REF** at (203.8, 109.5)
- removed the REF** at (126.0, 78.4)
- removed the REF** at (149.9, 138.4)
- removed the REF** at (147.8, 138.4)
- removed the REF** at (128.0, 140.5)
- removed the REF** at (133.8, 146.7)
- removed the REF** at (189.5, 119.3)
- removed the REF** at (188.5, 118.4)
- removed the REF** at (189.0, 118.9)
- removed the REF** at (192.7, 117.0)
- removed the REF** at (119.9, 86.6)
- removed the REF** at (133.7, 123.7)
- removed the REF** at (200.7, 150.4)
- removed the REF** at (200.7, 74.0)
- removed the REF** at (119.0, 150.4)
- removed the REF** at (119.0, 74.0)
- removed the REF** at (191.8, 123.7)
- removed the REF** at (191.8, 97.7)
- removed the REF** at (133.8, 97.7)
- removed the REF** at (191.8, 146.7)
- removed the REF** at (200.4, 127.8)
- removed the REF** at (124.0, 87.4)
- removed the REF** at (201.2, 127.8)
- removed the REF** at (201.9, 127.8)
- removed the REF** at (200.4, 130.0)
- removed the REF** at (201.2, 130.0)
- removed the REF** at (201.9, 130.0)
- removed the REF** at (191.1, 117.0)
- removed the REF** at (191.9, 117.0)
- removed the REF** at (124.0, 140.5)
- removed the REF** at (119.9, 87.4)
- removed the REF** at (203.8, 107.3)
- removed the REF** at (204.7, 107.3)
- removed the REF** at (205.4, 107.3)
- removed the REF** at (205.4, 109.5)
- removed the REF** at (204.7, 109.5)
- added R6: R, Resistor_SMD:R_1206_3216Metric_Pad1.42x1.75mm_HandSolder, F.Cu at (205.2, 105.7)
- added REF**: MountingHole_2.7mm_M2.5, MountingHole:MountingHole_2.7mm_M2.5, F.Cu at (119.0, 74.0)
- added REF**: MountingHole_2.7mm_M2.5, MountingHole:MountingHole_2.7mm_M2.5, F.Cu at (119.0, 150.4)
- added REF**: MountingHole_2.7mm_M2.5, MountingHole:MountingHole_2.7mm_M2.5, F.Cu at (200.7, 150.4)
- added REF**: MountingHole_2.7mm_M2.5, MountingHole:MountingHole_2.7mm_M2.5, F.Cu at (200.7, 74.0)
- added REF**: MountingHole_2.7mm_M2.5, MountingHole:MountingHole_2.7mm_M2.5, F.Cu at (126.0, 78.4)
- added REF**: MountingHole_2.7mm_M2.5, MountingHole:MountingHole_2.7mm_M2.5, F.Cu at (133.8, 97.7)
- added REF**: MountingHole_2.7mm_M2.5, MountingHole:MountingHole_2.7mm_M2.5, F.Cu at (191.8, 97.7)
- added REF**: MountingHole_2.7mm_M2.5, MountingHole:MountingHole_2.7mm_M2.5, F.Cu at (133.7, 123.7)
- added REF**: MountingHole_2.7mm_M2.5, MountingHole:MountingHole_2.7mm_M2.5, F.Cu at (191.8, 123.7)
- added REF**: MountingHole_2.7mm_M2.5, MountingHole:MountingHole_2.7mm_M2.5, F.Cu at (133.8, 146.7)
- added REF**: MountingHole_2.7mm_M2.5, MountingHole:MountingHole_2.7mm_M2.5, F.Cu at (191.8, 146.7)
- added U3: DHT11, Connector_PinHeader_2.54mm:PinHeader_1x04_P2.54mm_Vertical, F.Cu at (205.2, 111.8)
- added U7: LM2596_MODULE, regulators:LM2596_MODULE, F.Cu at (161.0, 88.4)
- moved R13 31.6 mm to (141.7, 117.3)
- moved Q5 31.3 mm to (147.3, 116.3)
- moved D5 31.1 mm to (146.3, 121.4)
- moved F1 27.2 mm to (149.4, 110.7), turned to 180 degrees
- moved D6 27.2 mm to (154.4, 105.2)
- moved U4 26.4 mm to (160.0, 94.5)
Connections:
- U1 pad 11: (no net) -> Net-(U1-Pad11)
- U1 pad 13: (no net) -> Net-(U1-Pad13)
- U1 pad 15: (no net) -> DHT_IO
- U1 pad 16: (no net) -> Net-(U1-Pad16)
- U1 pad 18: (no net) -> Net-(U1-Pad18)
- U1 pad 26: (no net) -> Net-(U1-Pad26)
- U1 pad 27: (no net) -> Net-(U1-Pad27)
- U1 pad 28: (no net) -> Net-(U1-Pad28)
- U1 pad 33: (no net) -> Net-(U1-Pad33)
- U1 pad 35: (no net) -> Net-(U1-Pad35)
- U1 pad 37: (no net) -> Net-(U1-Pad37)
- U1 pad 6: (no net) -> Net-(U1-Pad6)
- U1 pad 7: (no net) -> Net-(U1-Pad7)
- U2 pad 10: (no net) -> Net-(U2-Pad10)
- U2 pad 11: (no net) -> Net-(U2-Pad11)
- U2 pad 18: (no net) -> Net-(U2-Pad18)
- U2 pad 2: (no net) -> Net-(U2-Pad2)
- U2 pad 23: (no net) -> Net-(U2-Pad23)
- U2 pad 25: (no net) -> Net-(U2-Pad25)
- U2 pad 26: (no net) -> Net-(U2-Pad26)
- U2 pad 4: (no net) -> Net-(U2-Pad4)
- U2 pad 6: (no net) -> Net-(U2-Pad6)
- U2 pad 7: (no net) -> Net-(U2-Pad7)
- U2 pad 8: (no net) -> Net-(U2-Pad8)
- U2 pad 9: (no net) -> Net-(U2-Pad9)
Routing:
- net DHT_IO: track 0.00 -> 84.3 mm
- net 5V: track 185.2 -> 210.3 mm, vias 0 -> 1
- net 3.3V: track 169.5 -> 182.3 mm
- net Net-(D6-Pad2): track 109.2 -> 96.9 mm
- net Net-(D6-Pad1): track 72.5 -> 65.1 mm
- net Net-(J5-Pad1): track 63.6 -> 56.9 mm
- net GND: track 38.7 -> 43.3 mm, vias 0 -> 3
Other:
- outline, holes or cut-outs redrawn

Commit message: fan hole, space tunning
Parts:
- removed the REF** at (133.7, 123.7)
- added REF**: MountingHole_2.7mm_M2.5, MountingHole:MountingHole_2.7mm_M2.5, F.Cu at (176.0, 114.8)
- added REF**: MountingHole_2.7mm_M2.5, MountingHole:MountingHole_2.7mm_M2.5, F.Cu at (156.0, 114.8)
- added REF**: MountingHole_2.7mm_M2.5, MountingHole:MountingHole_2.7mm_M2.5, F.Cu at (156.0, 134.9)
- added REF**: MountingHole_2.7mm_M2.5, MountingHole:MountingHole_2.7mm_M2.5, F.Cu at (176.0, 134.9)
- added REF**: MountingHole_2.7mm_M2.5, MountingHole:MountingHole_2.7mm_M2.5, F.Cu at (126.0, 136.7)
- added REF**: MountingHole_2.7mm_M2.5, MountingHole:MountingHole_2.7mm_M2.5, F.Cu at (199.9, 81.7)
- U7: moved to B.Cu
- moved REF** 15.3 mm to (199.9, 136.7)
- moved D6 13.2 mm to (142.3, 99.9)
- moved U4 10.7 mm to (150.9, 89.0)
- moved F1 8.96 mm to (142.4, 105.2), turned to 0 degrees
- moved D5 8.18 mm to (140.7, 115.4)
- moved Q5 8.18 mm to (141.7, 110.4)
- moved R13 8.18 mm to (136.1, 111.4)
- moved REF** 4.90 mm to (199.9, 69.2)
- moved REF** 4.83 mm to (119.0, 69.2)
- moved R10 4.09 mm to (200.7, 130.2), turned to 180 degrees
- moved Q4 3.81 mm to (188.0, 83.8)
- moved D4 3.68 mm to (195.6, 90.2)
- moved U2 3.41 mm to (163.0, 109.3)
- moved REF** 3.27 mm to (126.0, 81.7)
- moved J7 2.67 mm to (198.9, 144.8)
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Routing:
- net GND: track 43.3 -> 81.5 mm, vias 3 -> 4
- net Net-(D6-Pad1): track 65.1 -> 75.9 mm, vias 0 -> 1
- net Net-(D6-Pad2): track 96.9 -> 88.9 mm
- net GPS_RST: track 13.1 -> 9.89 mm
- net CLK: track 18.1 -> 15.0 mm
- net MISO: track 18.1 -> 15.0 mm
- net MOSI: track 18.1 -> 15.0 mm
- net 5V: track 210.3 -> 213.2 mm, vias 1 -> 0
- net Net-(J5-Pad1): track 56.9 -> 59.7 mm
- net GPS_SUP: track 8.87 -> 6.35 mm
- net CE0: track 49.6 -> 47.4 mm
- net IC880A_RST: track 55.7 -> 53.5 mm
- net LED1: track 31.6 -> 33.5 mm
- net Net-(D4-Pad2): track 25.1 -> 26.6 mm
- net SCL: track 115.1 -> 116.4 mm
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Other:
- board size 93.9 x 83.8 mm -> 93.9 x 88.4 mm

Commit message: minor tunning
Parts:
- moved U4 1.78 mm to (149.1, 89.0)
Routing:
- net IC880A_RST: track 53.5 -> 12.0 mm
- net CE0: track 47.4 -> 26.0 mm
- net Net-(J5-Pad1): track 59.7 -> 64.3 mm
- net Net-(D6-Pad2): track 88.9 -> 91.6 mm
- net GND: track 81.5 -> 83.5 mm
- net 3.3V: track 183.1 -> 182.5 mm
- net Net-(D6-Pad1): track 75.9 -> 76.4 mm
Other:
- board text added: "coredump.ch CIT SU, FEI VSB 2019 https://lora.vsb.cz/"
- board text added: "iC880A Backplane v2.1-1"
- board text removed: "coredump.ch 2019"
- board text removed: "https://github.com/dbrgn/ic880a-backplane Designed in Switzerland"
- board text removed: "iC880A Backplane v2.1"

Commit message: Added texts, ground vias and minor tuning. This version 2.1-1 ready for prototyping
Parts:
- added REF**: VIA-0.6mm, StitchingVia:VIA-0.6mm, F.Cu at (123.4, 104.8)
- added REF**: VIA-0.6mm, StitchingVia:VIA-0.6mm, F.Cu at (202.7, 117.5)
- added REF**: VIA-0.6mm, StitchingVia:VIA-0.6mm, F.Cu at (202.7, 102.9)
- added REF**: VIA-0.6mm, StitchingVia:VIA-0.6mm, F.Cu at (191.4, 137.8)
- added REF**: VIA-0.6mm, StitchingVia:VIA-0.6mm, F.Cu at (194.7, 143.9)
- added REF**: VIA-0.6mm, StitchingVia:VIA-0.6mm, F.Cu at (142.0, 126.2)
- added REF**: VIA-0.6mm, StitchingVia:VIA-0.6mm, F.Cu at (175.6, 90.8)
- added REF**: VIA-0.6mm, StitchingVia:VIA-0.6mm, F.Cu at (205.2, 140.1)
- added REF**: VIA-0.6mm, StitchingVia:VIA-0.6mm, F.Cu at (133.0, 88.9)
- added REF**: VIA-0.6mm, StitchingVia:VIA-0.6mm, F.Cu at (123.4, 79.0)
- added REF**: VIA-0.6mm, StitchingVia:VIA-0.6mm, F.Cu at (118.6, 86.5)
- added REF**: VIA-0.6mm, StitchingVia:VIA-0.6mm, F.Cu at (119.1, 146.2)
- added REF**: VIA-0.6mm, StitchingVia:VIA-0.6mm, F.Cu at (205.4, 150.4)
- added REF**: VIA-0.6mm, StitchingVia:VIA-0.6mm, F.Cu at (205.4, 69.3)
Changed lines of the file:
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@@
     (tracks 431)
     (zones 0)
-    (modules 53)
+    (modules 67)
     (nets 57)
   )
   (page A4)
   (title_block
-    (title "iC880A-SPI Raspberry Pi Backplane")
-    (date 2019-07-16)
-    (rev v2.1)
-    (company "Coredump Rapperswil")
+    (title "iC880A Raspberry Pi Backplane")
+    (date 2019-08-22)
+    (rev v2.1-1)
+    (company "Coredump Rapperswil, https://coredump.ch")
+    (comment 1 "Modified by Jiri Slezka / CIT SU")
+    (comment 2 https://lora.vsb.cz)
   )
   (layers
@@
     (mod_text_size 1 1)
     (mod_text_width 0.15)
-    (pad_size 3 4)
-    (pad_drill 0.762)
+    (pad_size 0.6 0.6)
+    (pad_drill 0.4)
     (pad_to_mask_clearance 0.2)
     (solder_mask_min_width 0.25)
@@
     (visible_elements FFFFFF7F)
     (pcbplotparams
-      (layerselection 0x010fc_ffffffff)
+      (layerselection 0x010f0_ffffffff)
       (usegerberextensions true)
       (usegerberattributes false)
@@
       (drillshape 0)
       (scaleselection 1)
-      (outputdirectory "v2.1/"))
+      (outputdirectory "v2.1-1/"))
   )
   (net 0 "")
@@
     (add_net "Net-(Q5-Pad1)")
   )
+  (module StitchingVia:VIA-0.6mm (layer F.Cu)
+    (at 123.444 104.775)
+    (fp_text reference REF** (at 0 1.27) (layer F.SilkS) hide
+      (effects (font (size 1 1) (thickness 0.15)))
+    )
+    (fp_text value VIA-0.6mm (at 0 -1.27) (layer F.Fab) hide
+      (effects (font (size 1 1) (thickness 0.15)))
+    )
+    (pad 1 thru_hole circle (at 0 0) (size 0.6 0.6) (drill 0.4) (layers *.Cu)
+      (net 4 GND) (zone_connect 2))
+  )
+  (module StitchingVia:VIA-0.6mm (layer F.Cu)
+    (at 141.986 126.238)
+    (fp_text reference REF** (at 0 1.27) (layer F.SilkS) hide
+      (effects (font (size 1 1) (thickness 0.15)))
+    )
+    (fp_text value VIA-0.6mm (at 0 -1.27) (layer F.Fab) hide
+      (effects (font (size 1 1) (thickness 0.15)))
+    )
+    (pad 1 thru_hole circle (at 0 0) (size 0.6 0.6) (drill 0.4) (layers *.Cu)
+      (net 4 GND) (zone_connect 2))
+  )
+  (module StitchingVia:VIA-0.6mm (layer F.Cu)
+    (at 175.641 90.805)
+    (fp_text reference REF** (at 0 1.27) (layer F.SilkS) hide
+      (effects (font (size 1 1) (thickness 0.15)))
+    )
+    (fp_text value VIA-0.6mm (at 0 -1.27) (layer F.Fab) hide
+      (effects (font (size 1 1) (thickness 0.15)))
+    )
+    (pad 1 thru_hole circle (at 0 0) (size 0.6 0.6) (drill 0.4) (layers *.Cu)
+      (net 4 GND) (zone_connect 2))
+  )
+  (module StitchingVia:VIA-0.6mm (layer F.Cu)
+    (at 132.969 88.9)
+    (fp_text reference REF** (at 0 1.27) (layer F.SilkS) hide
+      (effects (font (size 1 1) (thickness 0.15)))
+    )
+    (fp_text value VIA-0.6mm (at 0 -1.27) (layer F.Fab) hide
+      (effects (font (size 1 1) (thickness 0.15)))
+    )
+    (pad 1 thru_hole circle (at 0 0) (size 0.6 0.6) (drill 0.4) (layers *.Cu)
+      (net 4 GND) (zone_connect 2))
+  )
+  (module StitchingVia:VIA-0.6mm (layer F.Cu)
+    (at 123.444 78.994)
+    (fp_text reference REF** (at 0 1.27) (layer F.SilkS) hide
+      (effects (font (size 1 1) (thickness 0.15)))
+    )
+    (fp_text value VIA-0.6mm (at 0 -1.27) (layer F.Fab) hide
+      (effects (font (size 1 1) (thickness 0.15)))
+    )
+    (pad 1 thru_hole circle (at 0 0) (size 0.6 0.6) (drill 0.4) (layers *.Cu)
+      (net 4 GND) (zone_connect 2))
+  )
+  (module StitchingVia:VIA-0.6mm (layer F.Cu)
+    (at 118.618 86.487)
+    (fp_text reference REF** (at 0 1.27) (layer F.SilkS) hide
+      (effects (font (size 1 1) (thickness 0.15)))
+    )
+    (fp_text value VIA-0.6mm (at 0 -1.27) (layer F.Fab) hide
+      (effects (font (size 1 1) (thickness 0.15)))
+    )
+    (pad 1 thru_hole circle (at 0 0) (size 0.6 0.6) (drill 0.4) (layers *.Cu)
+      (net 4 GND) (zone_connect 2))
+  )
+  (module StitchingVia:VIA-0.6mm (layer F.Cu)
+    (at 119.126 146.177)
+    (fp_text reference REF** (at 0 1.27) (layer F.SilkS) hide
+      (effects (font (size 1 1) (thickness 0.15)))
+    )
+    (fp_text value VIA-0.6mm (at 0 -1.27) (layer F.Fab) hide
+      (effects (font (size 1 1) (thickness 0.15)))
+    )
+    (pad 1 thru_hole circle (at 0 0) (size 0.6 0.6) (drill 0.4) (layers *.Cu)
+      (net 4 GND) (zone_connect 2))
+  )
+  (module StitchingVia:VIA-0.6mm (layer F.Cu)
+    (at 205.359 150.368)
+    (fp_text reference REF** (at 0 1.27) (layer F.SilkS) hide
+      (effects (font (size 1 1) (thickness 0.15)))
+    )
+    (fp_text value VIA-0.6mm (at 0 -1.27) (layer F.Fab) hide
+      (effects (font (size 1 1) (thickness 0.15)))
+    )
+    (pad 1 thru_hole circle (at 0 0) (size 0.6 0.6) (drill 0.4) (layers *.Cu)
+      (net 4 GND) (zone_connect 2))
+  )
+  (module StitchingVia:VIA-0.6mm (layer F.Cu)
+    (at 205.359 69.342)
+    (fp_text reference REF** (at 0 1.27) (layer F.SilkS) hide
+      (effects (font (size 1 1) (thickness 0.15)))
+    )
+    (fp_text value VIA-0.6mm (at 0 -1.27) (layer F.Fab) hide
+      (effects (font (size 1 1) (thickness 0.15)))
+    )
+    (pad 1 thru_hole circle (at 0 0) (size 0.6 0.6) (drill 0.4) (layers *.Cu)
+      (net 4 GND) (zone_connect 2))
+  )
+  (module StitchingVia:VIA-0.6mm (layer F.Cu)
+    (at 202.692 117.475)
+    (fp_text reference REF** (at 0 1.27) (layer F.SilkS) hide
+      (effects (font (size 1 1) (thickness 0.15)))
+    )
+    (fp_text value VIA-0.6mm (at 0 -1.27) (layer F.Fab) hide
+      (effects (font (size 1 1) (thickness 0.15)))
+    )
+    (pad 1 thru_hole circle (at 0 0) (size 0.6 0.6) (drill 0.4) (layers *.Cu)
+      (net 4 GND) (zone_connect 2))
+  )
+  (module StitchingVia:VIA-0.6mm (layer F.Cu)
+    (at 202.692 102.87)
+    (fp_text reference REF** (at 0 1.27) (layer F.SilkS) hide
+      (effects (font (size 1 1) (thickness 0.15)))
+    )
+    (fp_text value VIA-0.6mm (at 0 -1.27) (layer F.Fab) hide
+      (effects (font (size 1 1) (thickness 0.15)))
+    )
+    (pad 1 thru_hole circle (at 0 0) (size 0.6 0.6) (drill 0.4) (layers *.Cu)
+      (net 4 GND) (zone_connect 2))
+  )
+  (module StitchingVia:VIA-0.6mm (layer F.Cu)
+    (at 191.389 137.795)
+    (fp_text reference REF** (at 0 1.27) (layer F.SilkS) hide
+      (effects (font (size 1 1) (thickness 0.15)))
+    )
+    (fp_text value VIA-0.6mm (at 0 -1.27) (layer F.Fab) hide
+      (effects (font (size 1 1) (thickness 0.15)))
+    )
+    (pad 1 thru_hole circle (at 0 0) (size 0.6 0.6) (drill 0.4) (layers *.Cu)
+      (net 4 GND) (zone_connect 2))
+  )
+  (module StitchingVia:VIA-0.6mm (layer F.Cu)
+    (at 194.691 143.891)
+    (fp_text reference REF** (at 0 1.27) (layer F.SilkS) hide
+      (effects (font (size 1 1) (thickness 0.15)))
+    )
+    (fp_text value VIA-0.6mm (at 0 -1.27) (layer F.Fab) hide
+      (effects (font (size 1 1) (thickness 0.15)))
+    )
+    (pad 1 thru_hole circle (at 0 0) (size 0.6 0.6) (drill 0.4) (layers *.Cu)
+      (net 4 GND) (zone_connect 2))
+  )
   (module ic880a:IC880A-SPI (layer F.Cu)
     (at 162.9791 109.304)
@@
       (net 25 "Net-(D6-Pad1)"))
   )
+  (module StitchingVia:VIA-0.6mm (layer F.Cu)
+    (at 205.232 140.081)
+    (fp_text reference REF** (at 0 1.27) (layer F.SilkS) hide
+      (effects (font (size 1 1) (thickness 0.15)))
+    )
+    (fp_text value VIA-0.6mm (at 0 -1.27) (layer F.Fab) hide
+      (effects (font (size 1 1) (thickness 0.15)))
+    )
+    (pad 1 thru_hole circle (at 0 0) (size 0.6 0.6) (drill 0.4) (layers *.Cu)
+      (net 4 GND) (zone_connect 2))
+  )
   (gr_arc (start 166.497 86.995) (end 165.354 86.995) (angle -180) (layer Edge.Cuts) (width 0.15))

Commit message: verze 2.1-2
Parts:
- removed the REF** at (176.0, 114.8)
- removed the REF** at (156.0, 114.8)
- removed the REF** at (156.0, 134.9)
- removed the REF** at (176.0, 134.9)
- added REF**: MountingHole_2.7mm_M2.5, MountingHole:MountingHole_2.7mm_M2.5, F.Cu at (178.0, 116.8)
- added REF**: MountingHole_2.7mm_M2.5, MountingHole:MountingHole_2.7mm_M2.5, F.Cu at (158.0, 116.8)
- added REF**: MountingHole_2.7mm_M2.5, MountingHole:MountingHole_2.7mm_M2.5, F.Cu at (158.0, 136.9)
- added REF**: MountingHole_2.7mm_M2.5, MountingHole:MountingHole_2.7mm_M2.5, F.Cu at (178.0, 136.9)
- moved REF** 2.16 mm to (189.2, 137.8)
- moved U4 1.41 mm to (150.1, 90.0)
- moved U2 1.02 mm to (163.0, 110.3)
Routing:
- net GND: track 83.5 -> 53.8 mm
- net FAN: track 86.7 -> 80.0 mm
- net SCL: track 116.4 -> 112.4 mm
- net Net-(J5-Pad1): track 64.3 -> 61.0 mm
- net SDA: track 122.1 -> 118.8 mm
- net 5V: track 213.2 -> 215.2 mm
- net GPS_SUP: track 6.35 -> 4.44 mm
- net 3.3V: track 182.5 -> 180.8 mm
- net PPS: track 17.5 -> 16.1 mm
- net Net-(D6-Pad1): track 76.4 -> 75.2 mm
- net Net-(D6-Pad2): track 91.6 -> 92.5 mm
- net CE0: track 26.0 -> 25.5 mm
Other:
- outline, holes or cut-outs redrawn
- board text added: "iC880A Backplane v2.1-2"
- board text removed: "iC880A Backplane v2.1-1"

Commit message: added serial link to gps module on ic880a
Parts:
- added JP1: SolderJumper_2_Open, Jumper:SolderJumper-2_P1.3mm_Open_TrianglePad1.0x1.5mm, B.Cu at (184.8, 130.9)
- added JP2: SolderJumper_2_Open, Jumper:SolderJumper-2_P1.3mm_Open_TrianglePad1.0x1.5mm, B.Cu at (182.1, 130.9)
- added REF**: VIA-0.6mm, StitchingVia:VIA-0.6mm, F.Cu at (169.2, 100.6)
- added REF**: VIA-0.6mm, StitchingVia:VIA-0.6mm, F.Cu at (125.1, 68.8)
- added REF**: VIA-0.6mm, StitchingVia:VIA-0.6mm, F.Cu at (191.1, 123.8)
- added REF**: VIA-0.6mm, StitchingVia:VIA-0.6mm, F.Cu at (183.4, 133.9)
- C1, C3: value C -> 100nF; footprint Capacitors_SMD:C_1206 -> Capacitor_SMD:C_1206_3216Metric_Pad1.42x1.75mm_HandSolder
- D1, D2, D3: footprint LEDs:LED_1206 -> LED_SMD:LED_1206_3216Metric_Pad1.42x1.75mm_HandSolder
- D4, D6: value D -> SS14; footprint DO214:DO-214AC -> Diode_SMD:D_2114_3652Metric
- D5: value D_TVS -> TVSD SMBJ5.0A; footprint DO214:DO-214AA -> Diode_SMD:D_2114_3652Metric
- F1: value Polyfuse -> PolySwitch (PTC); footprint Capacitors_SMD:C_1812 -> Capacitor_SMD:C_1812_4532Metric_Pad1.30x3.40mm_HandSolder
- J4, J5: footprint Connectors_Terminal_Blocks:TerminalBlock_Pheonix_MPT-2.54mm_2pol -> TerminalBlock_Phoenix:TerminalBlock_Phoenix_MPT-0,5-2-2.54_1x02_P2.54mm_Horizontal
- J6: footprint headers:header_1x2_marked -> headers:header_1x2_unmarked
- Q4, Q5: footprint TO_SOT_Packages_SMD:SOT-23 -> Package_TO_SOT_SMD:SOT-23
- R1, R2, R3: footprint Resistors_SMD:R_1206 -> Resistor_SMD:R_1206_3216Metric_Pad1.42x1.75mm_HandSolder
- R10: value R -> 6.8kΩ; footprint Resistors_SMD:R_0805 -> Resistor_SMD:R_0805_2012Metric_Pad1.15x1.40mm_HandSolder
- R11: value R -> 3.6kΩ; footprint Resistors_SMD:R_0805 -> Resistor_SMD:R_0805_2012Metric_Pad1.15x1.40mm_HandSolder
- R12: value R -> 470Ω; footprint Resistors_SMD:R_0805 -> Resistor_SMD:R_0805_2012Metric_Pad1.15x1.40mm_HandSolder
- R13, R4, R5, R9: value R -> 10kΩ; footprint Resistors_SMD:R_1206 -> Resistor_SMD:R_1206_3216Metric_Pad1.42x1.75mm_HandSolder
- R6: value R -> 4.7kΩ
- U1: footprint headers:Pin_Header_Straight_2x20_Pitch2.54mm -> Connector_PinHeader_2.54mm:PinHeader_2x20_P2.54mm_Vertical
- U3: value DHT11 -> DHT22
- U5: footprint TO_SOT_Packages_SMD:SOT-23-6 -> Package_TO_SOT_SMD:SOT-23-6_Handsoldering
- moved REF** 9.02 mm to (118.6, 97.2)
- moved REF** 6.39 mm to (118.6, 74.8)
- moved REF** 3.58 mm to (118.7, 142.6)
- moved REF** 2.51 mm to (143.8, 128.0)
- moved REF** 1.88 mm to (177.3, 89.9)
- moved REF** 1.35 mm to (133.9, 89.9)
- moved J4 0.71 mm to (119.4, 90.0)
- moved J5 0.71 mm to (119.4, 80.2)
- moved REF** 0.52 mm to (205.2, 68.8)
Routing:
- net Net-(JP2-Pad1): track 0.00 -> 52.5 mm
- net Net-(JP1-Pad1): track 0.00 -> 52.5 mm
- net RX: track 30.8 -> 49.8 mm, vias 0 -> 1
- net TX: track 28.9 -> 47.6 mm, vias 0 -> 1
- net SCL: track 112.4 -> 115.5 mm
- net Net-(D6-Pad1): track 75.2 -> 76.1 mm
- net Net-(D6-Pad2): track 92.5 -> 91.9 mm
- net SDA: track 118.8 -> 118.2 mm
- net GND: vias 4 -> 3
